Commit message: gazebo

File: minesweeper_description/urdf/minesweeper.urdf.xacro (robot description, xacro)
@@ -3,10 +3,9 @@
     <xacro:arg name="robot_namespace" default="/" />
     <xacro:include filename="$(find minesweeper_description)/urdf/wheel.urdf.xacro"/>
-    <link
-      name="base_link">
+    <link name="base_link">
       <inertial>
-        <origin xyz="-0.00054987 4.6355E-06 0.05045" rpy="0 0 0" />
+        <origin xyz="0.0 0.0 0.05045" rpy="0 0 0" />
         <mass value="23.176" />
-        <inertia ixx="0.51234" ixy="0.0011009" ixz="-1.5952E-05" iyy="0.43777" iyz="-4.7203E-06" izz="0.9102"/>
+        <inertia ixx="0.6022" ixy="-0.02364" ixz="-0.1197" iyy="1.7386" iyz="-0.001544" izz="2.0296" />
       </inertial>
       <visual>
@@ -22,4 +21,5 @@
           <box size="0.75 0.50 0.15"/>
         </geometry>
+        <origin xyz="0.0 0.0 0.075"/>
       </collision>
     </link>

File: minesweeper_description/urdf/wheel.urdf.xacro (robot description, xacro)
@@ -14,5 +14,5 @@
           <collision>
               <geometry>
-                  <cylinder radius="0.17" length="0.11"/>
+                  <cylinder radius="0.165" length="0.11"/>
               </geometry>
               <origin xyz="0.0 0.0 0.0" rpy="0 ${radians(90)} ${radians(90)}"/>
@@ -24,4 +24,11 @@
           </inertial>
       </link>
+      <gazebo reference="${prefix}_wheel_link">
+  			<mu1 value="100.0"/>
+  			<mu2 value="50.0"/>
+  			<kp value="10000000.0" />
+  			<kd value="1.0" />
+  			<fdir1 value="1 0 0"/>
+  		</gazebo>
       <joint name="${prefix}_wheel" type="continuous">
           <parent link="base_link"/>
